Commit message: gripper control fixed

File: moveit_resources/panda_moveit_config/config/panda_arm_hand.srdf.xacro (robot description, xacro)
@@ -23,6 +23,6 @@
   </group_state>
   <group_state name="close" group="hand">
-    <joint name="panda_finger_joint1" value="0" />
-    <joint name="panda_finger_joint2" value="0" />
+    <joint name="panda_finger_joint1" value="0.02" />
+    <joint name="panda_finger_joint2" value="0.02" />
   </group_state>
   <!--END EFFECTOR: Purpose: Represent information about an end effector.-->
